File: V1/MCU.kicad_sch (KiCad schematic)
At the start: 9 parts, among them J2 Conn_01x08_Socket

Commit message: pcb design updated
Other:
- note added: "DRDY to MCU interrupt pin"
Changed lines of the file:
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@@
 	(generator_version "9.0")
 	(paper "A4")
+	(text "DRDY to MCU interrupt pin"
+		(exclude_from_sim no)
+		(at 233.172 73.406 0)
+		(effects
+			(font
+				(size 1.27 1.27)
+			)
+		)
+	)
 	(text "Progeamming_Connectors"
 		(exclude_from_sim no)
