File: V1/voltageRegulator.kicad_sch (KiCad schematic)
At the start: 23 parts, among them J3 Conn_01x02_Socket, U2 LT3045xMSE, U3 LM27762, U4 TP4056-42-ESOP8, U5 MIC5504-3.3YM5

Commit message: pcb design updated
Connections:
- no-connect marks 0 -> 1
Changed lines of the file:
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@@
 		(color 0 0 0 0)
 	)
+	(no_connect
+		(at 81.28 55.88)
+	)
 	(wire
 		(pts
@@
 	(polyline
 		(pts
-			(xy 11.43 85.09) (xy 284.48 85.09)
+			(xy 11.43 87.63) (xy 284.48 87.63)
 		)
 		(stroke
@@
 					(unit 1)
 				)
-			)
-		)
-	)
-	(symbol
-		(lib_id "power:+3.3V")
-		(at 276.86 60.96 0)
-		(unit 1)
-		(exclude_from_sim no)
-		(in_bom yes)
-		(on_board yes)
-		(dnp no)
-		(fields_autoplaced yes)
-		(property "Reference" "#PWR027"
-			(at 276.86 64.77 0)
-			(effects
-				(font
-					(size 1.27 1.27)
-				)
-				(hide yes)
-			)
-		)
-		(property "Value" "+3.3V"
-			(at 276.86 55.88 0)
-			(effects
-				(font
-					(size 1.27 1.27)
-				)
-			)
-		)
-		(property "Footprint" ""
-			(at 276.86 60.96 0)
-			(effects
-				(font
-					(size 1.27 1.27)
-				)
-				(hide yes)
-			)
-		)
-		(property "Datasheet" ""
-			(at 276.86 60.96 0)
-			(effects
-				(font
-					(size 1.27 1.27)
-				)
-				(hide yes)
-			)
-		)
-		(property "Description" "Power symbol creates a global label with name \"+3.3V\""
-			(at 276.86 60.96 0)
-			(effects
-				(font
-					(size 1.27 1.27)
-				)
-				(hide yes)
-			)
-		)
-		(pin "1"
-		)
-		(instances
-			(project ""
-				(path "/ed157c54-0048-40d2-ad12-afa32f500432/d8e482e9-881a-4209-91a3-a7fb6d3a9286"
-					(reference "#PWR027")
-					(unit 1)
-				)
