File: V1/V1.kicad_sch (KiCad schematic)
At the start: 20 parts, among them U1 ADS1299

Commit message: pcb design updated
Parts:
- added C20, C21: 1uF, Capacitor_SMD:C_0603_1608Metric_Pad1.08x0.95mm_HandSolder, symbol Device:C_Small
- added C22, C39: 10uF, Capacitor_SMD:C_0603_1608Metric_Pad1.08x0.95mm_HandSolder, symbol Device:C_Small
- added C23, C24: 1nF, Capacitor_SMD:C_0402_1005Metric, symbol Device:C_Small
- added C32: 0.47UF, Capacitor_SMD:C_0402_1005Metric, symbol Device:C_Small
- added C33: 4.7UF, Capacitor_SMD:C_0603_1608Metric, symbol Device:C_Small
- added C34: 10UF, Capacitor_SMD:C_0603_1608Metric, symbol Device:C_Small
- added C35, C40, C41: 10uF, Capacitor_SMD:C_0603_1608Metric, symbol Device:C_Small
- added C36, C37: 2.2uF, Capacitor_SMD:C_0603_1608Metric, symbol Device:C_Small
- added C38: 4.7uF, Capacitor_SMD:C_0603_1608Metric, symbol Device:C_Small
- added C42, C43: 1uF, Capacitor_SMD:C_0603_1608Metric, symbol Device:C_Small
- added D10, D2: LED, LED_SMD:LED_0603_1608Metric_Pad1.05x0.95mm_HandSolder, symbol Device:LED
- added J4: USB_C_Receptacle_PowerOnly_6P, Connector_USB:USB_C_Receptacle_GCT_USB4135-GF-A_6P_TopMnt_Horizontal, symbol Connector:USB_C_Receptacle_PowerOnly_6P
- added J5: Conn_01x08_Socket, Connector_PinHeader_2.54mm:PinHeader_1x08_P2.54mm_Vertical_SMD_Pin1Right, symbol Connector:Conn_01x08_Socket
- added J6: Conn_01x02_Socket, Connector_PinHeader_2.54mm:PinHeader_1x02_P2.54mm_Vertical, symbol Connector:Conn_01x02_Socket
- added NT1, NT2: NetTie_2, NetTie:NetTie-2_SMD_Pad0.5mm, symbol Device:NetTie_2
- added R10: 0.4R, Resistor_SMD:R_0603_1608Metric_Pad0.98x0.95mm_HandSolder, symbol Device:R_Small
- added R11, R12: 5.1k, Resistor_SMD:R_0603_1608Metric_Pad0.98x0.95mm_HandSolder, symbol Device:R_Small
- added R26, R27, R28, R29, R33, R35, R36: 10k, Resistor_SMD:R_0603_1608Metric_Pad0.98x0.95mm_HandSolder, symbol Device:R_Small
- added R30, R31, R32: 33R, Resistor_SMD:R_0603_1608Metric_Pad0.98x0.95mm_HandSolder, symbol Device:R_Small
- added R34: 25K, Resistor_SMD:R_0201_0603Metric_Pad0.64x0.40mm_HandSolder, symbol Device:R_Small
- added R37, R9: 1k, Resistor_SMD:R_0603_1608Metric_Pad0.98x0.95mm_HandSolder, symbol Device:R_Small
- added R38: 3k, Resistor_SMD:R_0603_1608Metric_Pad0.98x0.95mm_HandSolder, symbol Device:R_Small
- added TP1, TP2, TP3, TP4, TP5, TP6: TestPoint, TestPoint:TestPoint_Pad_1.0x1.0mm, symbol Connector:TestPoint
- added U2: REF5025AIDR, REF5025AIDR:SOIC-8_L4.9-W3.9-P1.27-LS6.0-BL, symbol REF5025AIDR:REF5025AIDR
- added U6: LT3045xMSE, Package_SO:MSOP-12-1EP_3x4.039mm_P0.65mm_EP1.651x2.845mm, symbol Regulator_Linear:LT3045xMSE
- added U7: LM27762, Package_SON:WSON-12-1EP_3x2mm_P0.5mm_EP1x2.65_ThermalVias, symbol Regulator_SwitchedCapacitor:LM27762
- added U8: TP4056-42-ESOP8, Package_SO:SOIC-8-1EP_3.9x4.9mm_P1.27mm_EP2.41x3.3mm_ThermalVias, symbol Battery_Management:TP4056-42-ESOP8
- added U9: MIC5504-3.3YM5, Package_TO_SOT_SMD:SOT-23-5, symbol Regulator_Linear:MIC5504-3.3YM5
- C1, C11, C12, C13, C14, C15, C16, C17, C2, C3, C4, C6, C7, C8, C9: footprint Capacitor_SMD:C_1206_3216Metric_Pad1.33x1.80mm_HandSolder -> Capacitor_SMD:C_0402_1005Metric
- C10, C5: footprint Capacitor_SMD:C_1206_3216Metric_Pad1.33x1.80mm_HandSolder -> Capacitor_SMD:C_0603_1608Metric
- C18, C19: footprint Capacitor_SMD:C_0603_1608Metric_Pad1.08x0.95mm_HandSolder -> Capacitor_SMD:C_0402_1005Metric
Connections:
- net +2V5: now also C34.2, TP5.1, U6.10 (OUTS), U6.11 (OUT), U6.12 (OUT)
- net +3.3V: now also C21.1, C43.1, R26.1, R27.1, R28.1, R29.1, R33.1, TP4.1, U2.2 (VIN), U9.5 (VOUT)
- net -2V5: now also C39.1, TP6.1, U7.6 (OUT-), U7.7 (FB-)
- net CS: now also J5.1 (Pin_1), R26.2
- net DIN: now also R31.1
- net DOUT: now also R32.1
- net DRDY: now also J5.2 (Pin_2), R27.2
- net GND: now also C23.1, C24.1, C40.2, C41.1, C42.2, C43.2, J4.A12 (GND), J4.B12 (GND), J4.S1 (SHIELD), J6.2 (Pin_2), NT1.2, NT2.1, R11.2, R12.2, R38.2, TP3.1, U7.12 (EN+), U8.1 (TEMP), U8.3 (GND), U8.9 (EPAD), U9.2 (GND); no longer C3.2, C4.2, U1.33 (DGND), U1.49 (DGND), U1.51 (DGND)
- net PWDN: now also J5.8 (Pin_8), R33.2
- net RESET: now also J5.6 (Pin_6), R28.2
- net SCLK: now also R30.1
- net START: now also J5.7 (Pin_7), R29.2
- net at C10.1, C11.1, U1.24 (VREFP): now also TP1.1
- net Electrode_4-: now reaches U1.1 (IN8N)
- net Electrode_4-: now also C24.2
- net Electrode_4+: now reaches U1.2 (IN8P)
- net Electrode_4+: now also C23.2
- new net: J5.5 (Pin_5), R31.2
- new net: J5.3 (Pin_3), R32.2
- new net: J5.4 (Pin_4), R30.2
- new net: R36.2, U7.8 (EN-)
- new net: J4.A5 (CC1), R11.1
- new net: J4.B5 (CC2), R12.1
- new net: C40.1, D10.2 (A), D2.2 (A), R10.1, U8.4 (V_{CC}), U8.8 (CE)
- new net: R35.2, U7.1 (PGOOD)
- new net: C36.1, U7.10 (C+)
- new net: C37.1, U7.11 (OUT+), U7.2 (FB+)
- new net: C38.1, U7.5 (CP)
- new net: C36.2, U7.9 (C-)
- new net: C20.1, U2.5 (TRIM/NR)
- new net: C22.1, TP2.1, U2.6 (VOUT)
- new net: R38.1, U8.2 (PROG)
- new net: R9.2, U8.6 (~{STDBY})
- new net: R37.2, U8.7 (~{CHRG})
- new net: D10.1 (K), R9.1
- new net: C32.1, R34.1, U6.8 (SET)
- new net: D2.1 (K), R37.1
- new net +BATT: C33.2, C35.1, C41.2, C42.1, J6.1 (Pin_1), R35.1, R36.1, U6.1 (IN), U6.2 (IN), U6.3 (IN), U6.4 (EN/UV), U6.7 (PGFB), U7.3 (VIN), U8.5 (BAT), U9.1 (VIN)
- new net GNDA: C20.2, C21.2, C22.2, C32.2, C33.1, C34.1, C35.2, C37.2, C38.2, C39.2, NT2.2, R34.2, U2.4 (GND), U6.13 (GND), U6.6 (ILIM), U6.9 (GND), U7.13 (PAD), U7.4 (GND)
- new net GNDD: C3.2, C4.2, NT1.1, U1.33 (DGND), U1.49 (DGND), U1.51 (DGND)
- new net VBUS: J4.A9 (VBUS), J4.B9 (VBUS), R10.2
- no-connect marks 0 -> 28
Other:
- removed sheet Electrode_connections
- removed sheet Programming_Connectors
- removed sheet Voltage_Regulator
- added sheet Electrodes_main_conn (Electrodes_mian.kicad_sch)
- note added: "+2.5V(AVDD)_Converter"
- note added: "-2.5V(AVSS)_Converter"
- note added: "3.3V_Converter (DVDD)"
- note added: "Battery_Connector"
- note added: "Charging_Module & Charge_Indicator"
- note added: "Connection_to_MCU"
- note added: "DRDY to MCU interrupt pin"
- note added: "STAR_Ground"
- note added: "USB_C_POWER"
- moved on the sheet: C1, C10, C11, C12, C13, C14, C15, C16, C17, C18, C19, C2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

Commit message: pcb design updated based on the suggestions.
Parts:
- added C45: 1.5nF, Capacitor_SMD:C_0402_1005Metric, symbol Device:C_Small
- added C46: 1nF, Capacitor_SMD:C_0402_1005Metric, symbol Device:C_Small
- added R13: 1M, Resistor_SMD:R_0805_2012Metric, symbol Device:R_Small_US
- C12, C13, C14, C15, C16, C17, C23, C24: value 1nF -> 10nF
Connections:
- net GND: now also C46.2
- net at U1.60 (BIASREF): now also C46.1
- net at U1.61 (BIASINV): now also C45.2, R13.2
- net at U1.63 (BIASOUT): now also C45.1, R13.1
- no-connect marks 28 -> 25
